Commit message: description: final assembly export — per-part structure with placeholder masses
- Re-export from pinned version URL (v/a87751ec): single arm chain, 8 DOF
  (mirror joints removed; dual motors are now separate parts inside links)
- Onshape materials provide placeholder mass/inertia on all links; measured
  values will override via link_masses.yaml
- postprocess: JOINT_RENAMES/LINK_RENAMES normalize export names
  (joint_2_main->joint_2, link1->link_1, link_2_holder->link_2, simple_6704->link_4)
- link_masses.yaml: scalar / shell+motors / parts+motors formats with
  parallel-axis composition (per-part weighing for carbon pipe + printed parts)
- tests updated to new assembly (43 passed)

File: description/arm_no_ee.urdf (robot description, URDF)
Before this commit: robot sopo, 7 links, 6 joints
Links:
- link link_1: mass 1e-09 -> 0.606896; geometry collision mesh filename=assets/joint_2_simple_sts3250__2_collision.stl; collision mesh filename=assets/joint_2_simple_sts3250_collision.stl
- link link_2: mass 1e-09 -> 0.626807; geometry collision mesh filename=assets/joint_3_simple_sts3250__2_collision.stl; collision mesh filename=assets/joint_3_simple_sts3250_collision.stl
- link link_3: mass 1e-09 -> 0.263483; geometry collision mesh filename=assets/joint_4_simple_sts3250_collision.stl; collision mesh filename=assets/link_3_collision.stl
- link link_4: mass 1e-09 -> 0.159854; geometry collision mesh filename=assets/joint_5_simple_sts3215_12v_collision.stl; collision mesh filename=assets/link_4_hold_1_collision.stl
- link link_5: mass 1e-09 -> 0.0810275; geometry collision mesh filename=assets/joint_6_simple_sts3215_12v_collision.stl; collision mesh filename=assets/link_5_collision.stl
- link sopo_desktop_base: mass 1e-09 -> 1.25391; geometry collision mesh filename=assets/simple61814_collision.stl; collision mesh filename=assets/simple_sm8512bl_collision.stl
Joints:
- joint joint_1: limit lower=-3.14159 upper=3.14159 effort=2.7 velocity=6.28 -> lower=-3.141592653589793 upper=3.141592653589793 effort=2.7 velocity=6.28; origin xyz=0 0.000980992 0.0777 rpy=3.14159 -0 0 -> xyz=-0 -0 0.0777 rpy=-3.14159 0 -0
- joint joint_2: origin xyz=-0 -0 -0.0412 rpy=1.5708 -0 -1.5708 -> xyz=-0.0185 0 -0.0412 rpy=1.5708 -0 -1.5708
- joint joint_3: limit lower=-1.5708 upper=1.6057 effort=3.1 velocity=7.85 -> lower=-1.5708 upper=1.5708 effort=3.1 velocity=7.85; origin xyz=5.48697e-07 -0.3429 -0 rpy=0 -0 0 -> xyz=5.48697e-07 -0.3428 -0 rpy=-0 -0 1.5708
- joint joint_4: limit lower=-3.12414 upper=3.12414 effort=1.6 velocity=7.85 -> lower=-3.14159 upper=3.14159 effort=1.6 velocity=7.85; origin xyz=-0.013 -0.0619 -0 rpy=-3.14159 1.5708 0 -> xyz=-0.0619 0.013 -0.0185 rpy=-1.5708 1.5708 0
- joint joint_5: origin xyz=-0 -4.74889e-07 -0.3726 rpy=0 -1.5708 0 -> xyz=0.0185 -9.39318e-07 -0.372226 rpy=3.14159 -1.5708 0
- joint joint_6: origin xyz=-0.0607257 -1.2e-11 -0 rpy=3.14159 -1.5708 0 -> xyz=-0.0611 1.2e-11 -0.0185 rpy=-0 1.5708 0

File: description/robot.urdf (robot description, URDF)
Before this commit: robot sopo, 9 links, 8 joints
Links:
- link ee: geometry collision mesh filename=assets/ee_collision.stl; collision mesh filename=assets/rod_d6_125.stl
- link link_1: mass 1e-09 -> 0.606896; geometry collision mesh filename=assets/joint_2_simple_sts3250__2_collision.stl; collision mesh filename=assets/joint_2_simple_sts3250_collision.stl
- link link_2: mass 1e-09 -> 0.626807; geometry collision mesh filename=assets/joint_3_simple_sts3250__2_collision.stl; collision mesh filename=assets/joint_3_simple_sts3250_collision.stl
- link link_3: mass 1e-09 -> 0.263483; geometry collision mesh filename=assets/joint_4_simple_sts3250_collision.stl; collision mesh filename=assets/link_3_collision.stl
- link link_4: mass 1e-09 -> 0.159854; geometry collision mesh filename=assets/joint_5_simple_sts3215_12v_collision.stl; collision mesh filename=assets/link_4_hold_1_collision.stl
- link link_5: mass 1e-09 -> 0.0810275; geometry collision mesh filename=assets/joint_6_simple_sts3215_12v_collision.stl; collision mesh filename=assets/link_5_collision.stl
- link sopo_desktop_base: mass 1e-09 -> 1.25391; geometry collision mesh filename=assets/simple61814_collision.stl; collision mesh filename=assets/simple_sm8512bl_collision.stl
Joints:
- joint joint_1: limit lower=-3.14159 upper=3.14159 effort=2.7 velocity=6.28 -> lower=-3.141592653589793 upper=3.141592653589793 effort=2.7 velocity=6.28; origin xyz=0 0.000980992 0.0777 rpy=3.14159 -0 0 -> xyz=-0 -0 0.0777 rpy=-3.14159 0 -0
- joint joint_2: origin xyz=-0 -0 -0.0412 rpy=1.5708 -0 -1.5708 -> xyz=-0.0185 0 -0.0412 rpy=1.5708 -0 -1.5708
- joint joint_3: limit lower=-1.5708 upper=1.6057 effort=3.1 velocity=7.85 -> lower=-1.5708 upper=1.5708 effort=3.1 velocity=7.85; origin xyz=5.48697e-07 -0.3429 -0 rpy=0 -0 0 -> xyz=5.48697e-07 -0.3428 -0 rpy=-0 -0 1.5708
- joint joint_4: limit lower=-3.12414 upper=3.12414 effort=1.6 velocity=7.85 -> lower=-3.14159 upper=3.14159 effort=1.6 velocity=7.85; origin xyz=-0.013 -0.0619 -0 rpy=-3.14159 1.5708 0 -> xyz=-0.0619 0.013 -0.0185 rpy=-1.5708 1.5708 0
- joint joint_5: origin xyz=-0 -4.74889e-07 -0.3726 rpy=0 -1.5708 0 -> xyz=0.0185 -9.39318e-07 -0.372226 rpy=3.14159 -1.5708 0
- joint joint_6: origin xyz=-0.0607257 -1.2e-11 -0 rpy=3.14159 -1.5708 0 -> xyz=-0.0611 1.2e-11 -0.0185 rpy=-0 1.5708 0
- joint left_finger_joint: origin xyz=0.0579601 -0.0159979 -0.063 rpy=-1.5708 -0 -1.5708 -> xyz=0.0579601 -0.0159979 -0.063 rpy=-1.5708 0 -1.5708
- joint right_finger_joint: origin xyz=-0.0580399 -0.0159979 -0.063 rpy=1.5708 -0 -1.5708 -> xyz=-0.0580399 -0.0159979 -0.063 rpy=1.5708 0 -1.5708

Commit message: dynamics: model-based gravity torque G(q) with hardware verification
- sopo/dynamics.py: pinocchio wrapper on arm_no_ee.urdf — gravity(q) [N·m],
  load_permille (stall-based duty prediction), external_torque (measured - G),
  extra_load_torque (known weight on flange, FK-exact lever), per-joint
  duty-to-torque scale support
- cookbook/17_gravity_check.py: interactive pose verification against
  Present_Load, --calibrate-vertical (URDF zero capture), --scale KG
  (hang known weight on flange, auto compute scale into calibration.yaml),
  dual-motor mounting-sign auto detection for error summary and ext estimate
- description/link_masses.yaml: measured arm link masses (per-part) injected;
  ee still estimate pending measurement
- calibration.yaml: gravity.zero_ticks / dir / scale (J2 0.289, J3 0.267, J5 0.236)
- verification on hardware: predicted vs measured loads converge within
  ~0.1 N·m per motor across poses; external torque near zero at free hold
- tests/test_dynamics.py: pinocchio vs pybullet cross-check (51 passed)

File: description/arm_no_ee.urdf (robot description, URDF)
Before this commit: robot sopo, 7 links, 6 joints
Links:
- link link_1: mass 0.606896 -> 1.239
- link link_2: mass 0.626807 -> 0.424
- link link_3: mass 0.263483 -> 0.1305
- link link_4: mass 0.159854 -> 0.307
- link link_5: mass 0.0810275 -> 0.087

File: description/robot.urdf (robot description, URDF)
Before this commit: robot sopo, 9 links, 8 joints
Links:
- link ee: mass 0.556 -> 0.522
- link link_1: mass 0.606896 -> 1.239
- link link_2: mass 0.626807 -> 0.424
- link link_3: mass 0.263483 -> 0.1305
- link link_4: mass 0.159854 -> 0.307
- link link_5: mass 0.0810275 -> 0.087

Commit message: description: REP-103 frame convention + stiff posing viewer
- base_link root (-90 deg z): approach direction is +x (REP-103 X fwd/Y left/Z up)
- axis flips: joint_1 yaw to +z (CCW from top), joint_4/joint_6 roll to approach
  (+x), joint_5 pitch aligned with joint_2/joint_3 (+y, +q leans forward)
  physical geometry/zero pose unchanged; sign convention only
- viewer model: drop actuator force limits, kp 2000 + damping 20 — sliders track
  immediately (was floppy due to real motor effort limits on posing actuators)
- cookbook/18_check_directions.py: per-joint jog to verify motor-tick vs URDF +q
  sign, writes calibration gravity.dir
- description/README.md: frame/joint-direction convention documented
- tests: 51 passed

File: description/arm_no_ee.urdf (robot description, URDF)
Before this commit: robot sopo, 7 links, 6 joints
Links:
- added link base_link, mass 1e-09
- link link_1: mass 1.239 -> 1.192
Joints:
- added joint base_fixed: type fixed, parent base_link, child sopo_desktop_base, origin xyz=0 0 0 rpy=0 0 -1.57079633
- joint joint_1: axis 0 0 1 -> 0 0 -1; limit lower=-3.141592653589793 upper=3.141592653589793 effort=2.7 velocity=6.28 -> lower=-3.14159265359 upper=3.14159265359 effort=2.7 velocity=6.28
- joint joint_4: axis 0 0 1 -> 0 0 -1
- joint joint_5: axis 0 0 1 -> 0 0 -1
- joint joint_6: axis 0 0 1 -> 0 0 -1

File: description/robot.urdf (robot description, URDF)
Before this commit: robot sopo, 9 links, 8 joints
Links:
- added link base_link, mass 1e-09
- link link_1: mass 1.239 -> 1.192
Joints:
- added joint base_fixed: type fixed, parent base_link, child sopo_desktop_base, origin xyz=0 0 0 rpy=0 0 -1.57079633
- joint joint_1: axis 0 0 1 -> 0 0 -1; limit lower=-3.141592653589793 upper=3.141592653589793 effort=2.7 velocity=6.28 -> lower=-3.14159265359 upper=3.14159265359 effort=2.7 velocity=6.28
- joint joint_4: axis 0 0 1 -> 0 0 -1
- joint joint_5: axis 0 0 1 -> 0 0 -1
- joint joint_6: axis 0 0 1 -> 0 0 -1
